Commit message: Updating anf syncing all files for ros_control on real_robot

File: urdf/depth_camera.xacro (robot description, xacro)
@@ -15,7 +15,7 @@
     </link>
     <joint name="camera_optical_joint" type="fixed">
-        <origin xyz="0 0 0" rpy="${-pi/2} 0 ${-pi/2}" />
         <parent link="camera_link" />
         <child link="camera_link_optical" />
+        <origin xyz="0 0 0" rpy="${-pi/2} 0 ${-pi/2}" />
     </joint>
     <link name="camera_link_optical"></link>

File: urdf/gazebo_control.xacro (robot description, xacro)
@@ -2,5 +2,4 @@
 <robot xmlns:xacro="http://www.ros.org/wiki/xacro">
     <gazebo>
-        <!-- Content will go here! -->
         <plugin name='diff_drive' filename='libgazebo_ros_diff_drive.so'>
             <!-- Wheel Information -->

File: urdf/robot_core.xacro (robot description, xacro)
@@ -2,18 +2,4 @@
 <robot xmlns:xacro="http://www.ros.org/wiki/xacro">
 	<xacro:include filename="inertial_macros.xacro" />
-	<!-- <xacro:property name="chassis_length" value="0.335"/>
-    <xacro:property name="chassis_width" value="0.265"/>
-    <xacro:property name="chassis_height" value="0.138"/>
-    <xacro:property name="chassis_mass" value="1.0"/>
-    <xacro:property name="wheel_radius" value="0.034"/>
-    <xacro:property name="wheel_thickness" value="0.026"/>
-    <xacro:property name="wheel_mass" value="0.05"/>
-    <xacro:property name="wheel_offset_x" value="0.226"/>
-    <xacro:property name="wheel_offset_y" value="0.166"/>
-    <xacro:property name="wheel_offset_z" value="0.01"/>
-    <xacro:property name="caster_wheel_radius" value="0.01"/>
-    <xacro:property name="caster_wheel_mass" value="0.01"/>
-    <xacro:property name="caster_wheel_offset_x" value="0.075"/>
-    <xacro:property name="caster_wheel_offset_z" value="${wheel_offset_z - wheel_radius + caster_wheel_radius}"/> -->
 	<xacro:property name="chassis_length" value="0.21"/>
     <xacro:property name="chassis_width" value="0.2"/>

Commit message: rtabmap_ros slam functionality added

File: urdf/depth_camera.xacro (robot description, xacro)
@@ -25,5 +25,5 @@
         <pose> 0 0 0 0 0 0 </pose>
         <visualize>true</visualize>
-        <update_rate>10</update_rate>
+        <update_rate>100</update_rate>
         <camera>
             <horizontal_fov>1.089</horizontal_fov>
@@ -40,4 +40,5 @@
         <plugin name="camera_controller" filename="libgazebo_ros_camera.so">
             <frame_name>camera_link_optical</frame_name>
+            <alwaysOn>true</alwaysOn>
             <min_depth>0.1</min_depth>
             <max_depth>100.0</max_depth>
@@ -45,3 +46,33 @@
     </sensor>
     </gazebo>
+    <!-- IMU Sensor Integration -->
+    <joint name="imu_joint" type="fixed">
+        <parent link="chassis"/>
+        <child link="imu_link"/>
+        <origin xyz="0.1 0 0.05" rpy="0 0 0"/>
+    </joint>
+    <link name="imu_link">
+        <visual>
+            <geometry>
+                <cylinder length="0.05" radius="0.02"/>
+            </geometry>
+            <material name="orange"/>
+        </visual>
+    </link>
+    <gazebo reference="imu_link">
+        <material>Gazebo/Orange</material>
+        <sensor name="imu_sensor" type="imu">
+            <pose>0 0 0 0 0 0</pose>
+            <update_rate>100</update_rate>
+            <imu>
+                <topic>/imu</topic>
+            </imu>
+            <plugin name="imu_plugin" filename="libgazebo_ros_imu_sensor.so">
+                <visualize>true</visualize>
+                <always_on>true</always_on>
+                <update_rate>100</update_rate>
+                <body_name>imu_link</body_name>
+            </plugin>
+        </sensor>
+    </gazebo>
 </robot>
